Commit message: changes to fuzzy controller and optimized fuzzy controller

File: src/gpg_urdf/urdf/description.xacro (robot description, xacro)
@@ -76,5 +76,5 @@
     <parent link="base_link"/>
     <child link="caster_wheel_link"/>
-    <origin xyz="-0.06 0 0.025" rpy="0 0 0" />
+    <origin xyz="-0.06 0 0.02" rpy="0 0 0" />
     <axis xyz="0 0 0"/>
   </joint>
@@ -82,5 +82,5 @@
     <visual>
       <geometry>
-        <sphere radius="0.025"/>
+        <sphere radius="0.02"/>
       </geometry>
       <origin rpy="0 0 0" xyz="0 0 0"/>
@@ -88,9 +88,9 @@
     <collision>
       <geometry>
-        <sphere radius="0.025"/>
+        <sphere radius="0.02"/>
       </geometry>
       <origin rpy="0 0 0" xyz="0 0 0"/>
     </collision>
-    <xacro:inertial_sphere mass="0.02" radius="0.025">
+    <xacro:inertial_sphere mass="0.02" radius="0.02">
       <origin rpy="0 0 0" xyz="0 0 0"/>
     </xacro:inertial_sphere>
